Commit message: wip

File: config/jaxa.urdf (robot description, URDF)
Before this commit: robot ivr, 57 links, 56 joints
Links:
- removed link grasp_link_1
- added link grasp_link
Joints:
- joint ARM1_GRASP: child grasp_link_1 -> grasp_link
- joint ARM1_GRIPPER: parent grasp_link_1 -> grasp_link

Commit message: updates for 5.0

File: config/jaxa.urdf (robot description, URDF)
Before this commit: robot ivr, 57 links, 56 joints
Links:
- removed link gripper_1
- added link gripper
Joints:
- joint ARM1_GRIPPER: child gripper_1 -> gripper
